Commit message: complete setup of world, robot and sensors

File: urdf/vlp16_l.urdf.xacro (robot description, xacro)
@@ -3,40 +3,101 @@
   <xacro:arg name="gpu" default="false"/>
   <xacro:property name="gpu" value="$(arg gpu)" />
+  <!-- define black color-->
   <material name="black">
     <color rgba="0 0 0 1"/>
   </material>
-  <!-- suporte -->
+  <!-- support link-->
   <link name="suport_link">
-    <inertial>
-      <origin xyz="0.0 0.0 0.0" rpy="0.0 0.0 0.0"/>
-      <mass value="1.0"/>
-      <inertia ixx="0.0" ixy="0.0" ixz="0.0" iyy="0.0" iyz="0.0" izz="0.0"/>
-    </inertial>
     <visual>
       <origin xyz="0.0 0.0 0.0" rpy="0.0 0.0 0.0"/>
       <geometry>
-        <cylinder radius="0.04" length="0.1"/>
+        <cylinder radius="0.045" length="0.08"/>
       </geometry>
-      <gazebo reference="black">
-        <material>Gazebo/Black</material>
-      </gazebo>
+      <material name="black"/>
     </visual>
     <collision>
       <origin xyz="0.0 0.0 0.0" rpy="0.0 0.0 0.0"/>
       <geometry>
-        <cylinder radius="0.04" length="0.1"/>
+        <cylinder radius="0.045" length="0.08"/>
       </geometry>
     </collision>
+    <inertial>
+      <origin xyz="0.0 0.0 0.0" rpy="0.0 0.0 0.0"/>
+      <mass value="0.1"/>
+      <inertia ixx="0.00010395833333333333" ixy="0.0" ixz="0.0" iyy="0.00010395833333333333" iyz="0.0" izz="0.00010125"/>
+    </inertial>
   </link>
+  <!-- black color reference for gazebo -->
+  <gazebo reference="suport_link">
+    <material>Gazebo/Black</material>
+  </gazebo>
+  <!-- joint between husky and support -->
   <joint name="husky_suport" type="fixed">
-    <origin xyz="0.0 0.0 0.05" rpy="0.0 0.0 0.0"/>
+    <origin xyz="0.0 0.0 0.04" rpy="0.0 0.0 0.0"/>
     <parent link="top_plate_link"/>
     <child link="suport_link"/>
   </joint>
-  <!-- velodyne lidar
+  <!-- velodyne lidar  and joint between lidar and suport -->
   <xacro:include filename="$(find velodyne_description)/urdf/VLP-16.urdf.xacro"/>
-  <VLP-16 parent="top_plate_link" name="velodyne" topic="/velodyne_points" hz="10" samples="440" gpu="${gpu}">
-    <origin xyz="0 0 2" rpy="0 0 0" />
-  </VLP-16> -->
-  <!-- Kinect camera -->
+  <VLP-16 parent="suport_link" name="velodyne" topic="/velodyne_points" hz="10" samples="440" gpu="${gpu}">
+    <origin xyz="0 0 0.04" rpy="0 0 0" />
+  </VLP-16>
+  <!-- kinect camera -->
+  <link name="kinect_link">
+    <visual>
+      <origin xyz="0.0 0.0 0.0" rpy="0.0 0.0 0.0"/>
+      <geometry>
+        <mesh filename="model://kinect/meshes/kinect.dae"/>
+      </geometry>
+    </visual>
+    <collision>
+      <origin xyz="0.0 0.0 0.0" rpy="0.0 0.0 0.0"/>
+      <geometry>
+        <mesh filename="model://kinect/meshes/kinect.dae"/>
+      </geometry>
+    </collision>
+    <inertial>
+      <origin xyz="0.0 0.0 0.0" rpy="0.0 0.0 0.0"/>
+      <mass value="0.1"/>
+      <inertia ixx="1.0" ixy="0.0" ixz="0.0" iyy="1.0" iyz="0.0" izz="1.0"/>
+    </inertial>
+  </link>
+  <!-- kinect camera plugin 720p-->
+  <gazebo reference="kinect_link">
+    <sensor type="camera" name="camera_top">
+      <update_rate>30.0</update_rate>
+      <camera name="head">
+        <horizontal_fov>1.3962634</horizontal_fov>
+        <image>
+          <width>1280</width>
+          <height>720</height>
+          <format>R8G8B8</format>
+        </image>
+        <clip>
+          <near>0.02</near>
+          <far>300</far>
+        </clip>
+      </camera>
+      <plugin name="camera_controller" filename="libgazebo_ros_camera.so">
+        <alwaysOn>true</alwaysOn>
+        <updateRate>0.0</updateRate>
+        <cameraName>diff/camera_top</cameraName>
+        <imageTopicName>image_raw</imageTopicName>
+        <cameraInfoTopicName>camera_info</cameraInfoTopicName>
+        <frameName>kinect_link</frameName>
+        <hackBaseline>0.07</hackBaseline>
+        <distortionK1>0.0</distortionK1>
+        <distortionK2>0.0</distortionK2>
+        <distortionK3>0.0</distortionK3>
+        <distortionT1>0.0</distortionT1>
+        <distortionT2>0.0</distortionT2>
+      </plugin>
+    </sensor>
+  </gazebo>
+  <!-- joint between kinect and lidar -->
+  <joint name="lidar_kinect" type="fixed">
+    <origin xyz="0.03 0.0 0.08" rpy="0.0 0.0 0.0"/>
+    <parent link="velodyne"/>
+    <child link="kinect_link"/>
+  </joint>
 </robot>
